File: phMeter.kicad_pcb (KiCad board)
At the start: 2 copper layers, 25.4 x 63.5 mm, 30 parts, among them J1 PH_PROBE, J2 QWIIC, J3 I2C, U1 LTC2471, U2 LMP7721, U3 ADM3260, U4 LMP7721, U5 MCP1501

Commit message: SCH REV B0, PCB REV B0
Parts:
- removed the C13 at (142.5, 99.6)
- removed RN1: MPMT2001AT1, Package_TO_SOT_SMD:SOT-23
- added C14: 0.1uF, Capacitor_Tantalum_SMD:CP_EIA-2012-15_AVX-P, F.Cu at (142.2, 98.6)
- added C7: 0.1uF, Capacitor_Tantalum_SMD:CP_EIA-2012-15_AVX-P, F.Cu at (151.4, 98.6)
- added R10: 10k, jlcpcb_smt:R_0603_1608Metric, F.Cu at (140.1, 88.9)
- added R4: 1k, jlcpcb_smt:R_0603_1608Metric, F.Cu at (147.1, 103.9)
- added R9: 10k, jlcpcb_smt:R_0603_1608Metric, F.Cu at (141.9, 88.9)
- added REF**: KiCad-Logo2_6mm_SilkScreen, Symbol:KiCad-Logo2_6mm_SilkScreen, F.Cu at (157.6, 102.4)
- C6: value 0.1uF -> 1uF
- U1: value LTC2471 -> LTC2473
- moved C6 8.18 mm to (144.3, 103.1)
- moved C3 2.16 mm to (143.5, 108.0)
- moved C2 1.98 mm to (145.3, 108.0)
- moved C15 0.92 mm to (141.0, 81.0)
- renumbered C2 to C1, C9 to C10, C10 to C11, C11 to C12, C12 to C13, C14 to C15, C3 to C2, C4 to C3, C5 to C4, C1 to C5, C7 to C8, C8 to C9, R4 to R5, R5 to R6, R6 to R7, R7 to R8
Connections:
- C6 pad 1: +3V3 -> /VREF
- U1 pad 10: GNDS -> Net-(R4-Pad1)
- U4 pad 1: Net-(RN1-Pad3) -> /VREF
- U5 pad 1: /VREF -> Net-(R9-Pad1)
Routing:
- net /VREF: track 3.91 -> 24.8 mm
- net /PROBE_V_OUT: track 58.6 -> 52.0 mm, vias 1 -> 2
- net Net-(R4-Pad1): track 0.00 -> 4.31 mm, vias 0 -> 1
- net Net-(R9-Pad1): track 0.00 -> 3.43 mm
- net Net-(RN1-Pad3): track 2.72 -> 0.00 mm
- net GNDS: track 36.3 -> 37.4 mm
- added copper zone on B.Cu, net /PROBE_V_OUT
Other:
- board text added: "A0 - Inital Revision B0 - Integrate changes from schematic REV B0, Add copper pour under guard ring on B.Cu Minor silkscreen changes"
- board text added: "Changelog"
- board text added: "pH Probe to isolated I2C circuit svcguy REV B0 06/2021"
- board text removed: "pH Probe to isolated I2C circuit svcguy REV A0 06/2021"

Commit message: SCH REV C0, PCB REV C0, added simulation files
Parts:
- C5, C6: value 1uF -> 0.1uF
- moved C5 3.66 mm to (150.1, 104.4), turned to 0 degrees
- moved REF** 3.22 mm to (159.5, 105.0), turned to 270 degrees
- moved C6 3.07 mm to (147.1, 104.4)
- moved R4 1.93 mm to (147.8, 102.1)
- moved R3 1.85 mm to (149.4, 102.1)
Connections:
- C5 pad 1: /PROBE_V_OUT -> Net-(C5-Pad1)
- C6 pad 1: /VREF -> Net-(C6-Pad1)
- R3 pad 1: Net-(R3-Pad1) -> Net-(C5-Pad1)
- R4 pad 1: Net-(R4-Pad1) -> Net-(C6-Pad1)
- U1 pad 10: Net-(R4-Pad1) -> Net-(C6-Pad1)
- U1 pad 9: Net-(R3-Pad1) -> Net-(C5-Pad1)
Routing:
- net /PROBE_V_OUT: track 52.0 -> 57.6 mm, vias 2 -> 3
- net Net-(C5-Pad1): track 0.00 -> 4.36 mm
- net Net-(C6-Pad1): track 0.00 -> 4.36 mm
- net Net-(R4-Pad1): track 4.31 -> 0.00 mm, vias 1 -> 0
- net Net-(R3-Pad1): track 2.43 -> 0.00 mm
Other:
- board text added: "A0 - Inital Revision B0 - Integrate changes from schematic REV B0, Add copper pour under guard ring on B.Cu Minor silkscreen changes C0 - Integrate chagnes from schematic REV C0, Minor silkscreen changes"
- board text added: "pH Probe to isolated I2C circuit svcguy REV C0 06/2021"
- board text removed: "A0 - Inital Revision B0 - Integrate changes from schematic REV B0, Add copper pour under guard ring on B.Cu Minor silkscreen changes"
- board text removed: "pH Probe to isolated I2C circuit svcguy REV B0 06/2021"
