File: phMeter.sch (KiCad schematic (older format))
At the start: 30 parts, among them J1 PH_PROBE, J2 QWIIC, J3 I2C, U1 LTC2471, U2 LMP7721, U3 ADM3260, U4 LMP7721, U5 MCP1501

Commit message: SCH REV B0, PCB REV B0
Parts:
- removed RN1: MPMT2001AT1, Package_TO_SOT_SMD:SOT-23, symbol Device:Voltage_Divider_CenterPin3
- removed U1: LTC2471, Package_SO:MSOP-12_3x4mm_P0.65mm, symbol Custom_KiCAD:LTC2471
- added C6: 1uF, jlcpcb_smt:C_0603_1608Metric, symbol Device:C
- added R10, R9: 10k, jlcpcb_smt:R_0603_1608Metric, symbol Device:R_US
- added R4: 1k, jlcpcb_smt:R_0603_1608Metric, symbol Device:R_US
- added U1: LTC2473, Package_SO:MSOP-12_3x4mm_P0.65mm, symbol Custom_KiCAD:LTC2473
- C14: renamed from C13; footprint jlcpcb_smt:C_0603_1608Metric -> Capacitor_Tantalum_SMD:CP_EIA-2012-15_AVX-P
- C15: renamed from C14; Digikey 445-5964-1-ND -> 445-6933-1-ND
- C7: renamed from C6; footprint jlcpcb_smt:C_0603_1608Metric -> Capacitor_Tantalum_SMD:CP_EIA-2012-15_AVX-P
- U3: Digikey (none) -> ADM3260ARSZ-RL7CT-ND
- U5: Digikey (none) -> MCP1501T-10E/CHYCT-ND
- renumbered C2 to C1, C9 to C10, C10 to C11, C11 to C12, C12 to C13, C3 to C2, C4 to C3, C5 to C4, C1 to C5, C7 to C8, C8 to C9, R4 to R5, R5 to R6, R6 to R7, R7 to R8
Connections:
- net +3V3: now also U1.12 (VCC)
- net GNDS: now also C6.2, R10.2, U1.11 (GND), U1.3 (A0), U1.4 (GND), U1.7 (GND), U1.8 (REF-)
- net SCL_ISO: now also U1.5 (SCL)
- net SDA_ISO: now also U1.6 (SDA)
- net VREF: now also U4.1 (IN+), C6.1, R10.1, R4.2, R9.2; no longer U5.1 (OUT)
- net at C1.1: now also U1.1 (REFOUT)
- net at C4.1: now also U1.2 (COMP)
- net at R3.1: now also U1.9 (IN+)
- new net: R9.1, U5.1 (OUT)
- new net: R4.1, U1.10 (IN-)
Other:
- note added: "1 - C7, C14 are low leakage tantalums, all others standard 0603 MLCC\n2 - R9, R10 are metal film 1% or better, R7, R8 are 1% or better, all others standard 0603\n3 - Guard ring trace should encircle high impedance trace on top side and have a copper fill \non bot side under high impedence trace\n4 - J1 is a BNC type connector, impedence not specified"
- note added: "A0 - Inital revision\nB0 - Fix LMP7721 symbols, replace VREF resistor network with\n discrete resistors, replace LTC2471 with LTC2473 and use\n VREF as IN-, add LPF to VREF"
- note added: "Changelog"
- note added: "Notes"
- moved on the sheet: C5, R3

Commit message: SCH REV C0, PCB REV C0, added simulation files
Parts:
- C5, C6: value 1uF -> 0.1uF; Digikey 478-8928-1-ND -> 311-1088-1-ND
Connections:
- net PROBE_V_OUT: no longer C5.1
- net VREF: no longer C6.1
- net at R4.1, U1.10 (IN-): now also C6.1
- net at R3.1, U1.9 (IN+): now also C5.1
Other:
- note added: "A0 - Inital revision\nB0 - Fix LMP7721 symbols, replace VREF resistor network with\n discrete resistors, replace LTC2471 with LTC2473 and use\n VREF as IN-, add LPF to VREF\nC0 - Change C5, C6 to 0.1uF according to LTC2473 datasheet,\n move C5, C6 closer to LTC2473, Add LTC2473 I2C address note\n"
- note added: "A0 = GND, I2C ADDRESS = 0x14"
- note removed: "A0 - Inital revision\nB0 - Fix LMP7721 symbols, replace VREF resistor network with\n discrete resistors, replace LTC2471 with LTC2473 and use\n VREF as IN-, add LPF to VREF"
- moved on the sheet: C5, R3, R4
Changed lines of the file:
@@
 Title "phMeter"
 Date "2021-06-07"
-Rev "B0"
+Rev "C0"
 Comp "svcguy"
 Comment1 ""
@@
 L Device:R_US R3
 U 1 1 60E8F4F8
-P 6350 1900
-F 0 "R3" V 6145 1900 50  0000 C CNN
-F 1 "1k" V 6236 1900 50  0000 C CNN
-F 2 "jlcpcb_smt:R_0603_1608Metric" V 6390 1890 50  0001 C CNN
-F 3 "~" H 6350 1900 50  0001 C CNN
-F 4 "P1.00KHCT-ND" H 6350 1900 50  0001 C CNN "Digikey"
-	1    6350 1900
+P 5700 1900
+F 0 "R3" V 5495 1900 50  0000 C CNN
+F 1 "1k" V 5586 1900 50  0000 C CNN
+F 2 "jlcpcb_smt:R_0603_1608Metric" V 5740 1890 50  0001 C CNN
+F 3 "~" H 5700 1900 50  0001 C CNN
+F 4 "P1.00KHCT-ND" H 5700 1900 50  0001 C CNN "Digikey"
+	1    5700 1900
 	0    1    1    0
 $EndComp
@@
 L Device:C C5
 U 1 1 60E90862
-P 6000 2450
-F 0 "C5" H 6115 2496 50  0000 L CNN
-F 1 "1uF" H 6115 2405 50  0000 L CNN
-F 2 "jlcpcb_smt:C_0603_1608Metric" H 6038 2300 50  0001 C CNN
-F 3 "~" H 6000 2450 50  0001 C CNN
-F 4 "478-8928-1-ND" H 6000 2450 50  0001 C CNN "Digikey"
-	1    6000 2450
-	1    0    0    -1
-$EndComp
-Wire Wire Line
-	6000 2600 6000 2650
-Wire Wire Line
-	6200 1900 6000 1900
-Wire Wire Line
-	6000 1900 6000 2300
-Wire Wire Line
-	6000 1900 5600 1900
-Connection ~ 6000 1900
-Text Label 5600 1900 2    50   ~ 0
+P 5950 2450
+F 0 "C5" H 6065 2496 50  0000 L CNN
+F 1 "0.1uF" H 6065 2405 50  0000 L CNN
+F 2 "jlcpcb_smt:C_0603_1608Metric" H 5988 2300 50  0001 C CNN
+F 3 "~" H 5950 2450 50  0001 C CNN
+F 4 "311-1088-1-ND" H 5950 2450 50  0001 C CNN "Digikey"
+	1    5950 2450
+	1    0    0    -1
+$EndComp
+Wire Wire Line
+	5950 2600 5950 2650
+Text Label 5400 1900 2    50   ~ 0
 PROBE_V_OUT
 Text Label 1900 4900 2    50   ~ 0
@@
 L power:GNDS #PWR03
 U 1 1 60C1ECC9
-P 6000 2650
-F 0 "#PWR03" H 6000 2400 50  0001 C CNN
-F 1 "GNDS" H 6005 2477 50  0000 C CNN
-F 2 "" H 6000 2650 50  0001 C CNN
-F 3 "" H 6000 2650 50  0001 C CNN
-	1    6000 2650
+P 5950 2650
+F 0 "#PWR03" H 5950 2400 50  0001 C CNN
+F 1 "GNDS" H 5955 2477 50  0000 C CNN
+F 2 "" H 5950 2650 50  0001 C CNN
+F 3 "" H 5950 2650 50  0001 C CNN
+	1    5950 2650
 	1    0    0    -1
 $EndComp
@@
 	7750 2650 8050 2650
 Wire Wire Line
-	7450 1900 6500 1900
+	7450 1900 5950 1900
 $Comp
 L Device:R_US R9
@@
 Wire Wire Line
 	1250 7100 1250 7150
-Text Label 5600 2000 2    50   ~ 0
+Text Label 5400 2000 2    50   ~ 0
 VREF
 $Comp
 L Device:R_US R4
 U 1 1 60C4F1FB
-P 6650 2000
-F 0 "R4" V 6750 2000 50  0000 C CNN
-F 1 "1k" V 6850 2000 50  0000 C CNN
-F 2 "jlcpcb_smt:R_0603_1608Metric" V 6690 1990 50  0001 C CNN
-F 3 "~" H 6650 2000 50  0001 C CNN
-F 4 "P1.00KHCT-ND" H 6650 2000 50  0001 C CNN "Digikey"
-	1    6650 2000
+P 6150 2000
+F 0 "R4" V 6250 2000 50  0000 C CNN
+F 1 "1k" V 6350 2000 50  0000 C CNN
+F 2 "jlcpcb_smt:R_0603_1608Metric" V 6190 1990 50  0001 C CNN
+F 3 "~" H 6150 2000 50  0001 C CNN
+F 4 "P1.00KHCT-ND" H 6150 2000 50  0001 C CNN "Digikey"
+	1    6150 2000
 	0    1    1    0
 $EndComp
 Wire Wire Line
-	5600 2000 6400 2000
-Wire Wire Line
-	6800 2000 7450 2000
+	6300 2000 6400 2000
 $Comp
 L Device:C C6
@@
 P 6400 2450
 F 0 "C6" H 6515 2496 50  0000 L CNN
-F 1 "1uF" H 6515 2405 50  0000 L CNN
+F 1 "0.1uF" H 6515 2405 50  0000 L CNN
 F 2 "jlcpcb_smt:C_0603_1608Metric" H 6438 2300 50  0001 C CNN
 F 3 "~" H 6400 2450 50  0001 C CNN
-F 4 "478-8928-1-ND" H 6400 2450 50  0001 C CNN "Digikey"
+F 4 "311-1088-1-ND" H 6400 2450 50  0001 C CNN "Digikey"
 	1    6400 2450
 	1    0    0    -1
 $EndComp
-Wire Wire Line
-	6400 2000 6400 2300
-Connection ~ 6400 2000
-Wire Wire Line
-	6400 2000 6500 2000
 $Comp
 L power:GNDS #PWR04
@@
 Text Notes 650  1200 0    50   ~ 0
 1 - C7, C14 are low leakage tantalums, all others standard 0603 MLCC\n2 - R9, R10 are metal film 1% or better,  R7, R8 are 1% or better, all others standard 0603\n3 - Guard ring trace should encircle high impedance trace on top side and have a copper fill \non bot side under high impedence trace\n4 - J1 is a BNC type connector, impedence not specified
-Text Notes 11800 800  0    50   ~ 0
-A0 - Inital revision\nB0 - Fix LMP7721 symbols, replace VREF resistor network with\n       discrete resistors, replace LTC2471 with LTC2473 and use\n       VREF as IN-, add LPF to VREF
+Text Notes 11800 950  0    50   ~ 0
+A0 - Inital revision\nB0 - Fix LMP7721 symbols, replace VREF resistor network with\n       discrete resistors, replace LTC2471 with LTC2473 and use\n       VREF as IN-, add LPF to VREF\nC0 - Change C5, C6 to 0.1uF according to LTC2473 datasheet,\n       move C5, C6 closer to LTC2473, Add LTC2473 I2C address note\n
 Text Notes 11800 400  0    100  Italic 20
 Changelog
+Text Notes 7150 3200 0    50   Italic 0
+A0 = GND, I2C ADDRESS = 0x14
+Wire Wire Line
+	5400 1900 5550 1900
+Wire Wire Line
+	5950 2300 5950 1900
+Connection ~ 5950 1900
+Wire Wire Line
+	5950 1900 5850 1900
+Wire Wire Line
+	5400 2000 6000 2000
+Wire Wire Line
+	6400 2300 6400 2000
+Connection ~ 6400 2000
+Wire Wire Line
+	6400 2000 7450 2000
 $EndSCHEMATC
